File: Rev_1/ECAD/board/Kicad/Filtering.kicad_sch (KiCad schematic)
At the start: 26 parts, among them U301 LM324, U302 LM324

Commit message: Added gain and rectifier stage
Parts:
- removed U? (x2): LM324, symbol Amplifier_Operational:LM324
- added unit 3 of U302
- added unit 4 of U302
Connections:
- net AUDIO OUT: now also U302.13 (-), U302.14
- net at C308.1, R309.1: now also U302.8, U302.9 (-)
- net at C307.2, R308.2: now also U302.10 (+)
- net at C309.2, R310.2: now also U302.12 (+)
